Commit message: No idea

File: common.urdf.xacro (robot description, xacro)
@@ -1,4 +1,7 @@
 <?xml version="1.0"?>
 <robot xmlns:xacro="http://www.ros.org/wiki/xacro">
+    <xacro:macro name="default_origin">
+        <origin rpy="0 0 0"/>
+    </xacro:macro>
     <xacro:macro name="rot_x_origin">
         <origin rpy="0 ${pi/2} 0"/>

File: joints.urdf.xacro (robot description, xacro)
@@ -1,5 +1,5 @@
 <?xml version="1.0"?>
 <robot xmlns:xacro="http://www.ros.org/wiki/xacro">
-    <xacro:macro name="rot_joint" params="parent child *origin *axis effort velocity damping">
+    <xacro:macro name="rot_joint" params="parent child effort velocity damping *origin *axis ">
         <joint name="${parent}_${child}_joint" type="revolute">
             <parent link="${parent}_link"/>

File: links.urdf.xacro (robot description, xacro)
@@ -1,4 +1,7 @@
 <?xml version="1.0"?>
 <robot xmlns:xacro="http://www.ros.org/wiki/xacro">
+    <xacro:macro name="world">
+        <link name="world"/>
+    </xacro:macro>
     <xacro:macro name="base">
         <link name="base_link"/>
